Commit message: ros_melodic
Funciona en ros Melodic

File: surfr_urx/urx_driver/urdf/ur3_robot.urdf.xacro (robot description, xacro)
@@ -8,5 +8,5 @@
   <!-- arm -->
   <xacro:ur3_robot prefix="$(arg prefix)/" joint_limited="false" tcp_position="$(arg tcp_position)" tcp_orientation="$(arg tcp_orientation)" />
-  <link name="$(arg origin_name)" />
+<link name="$(arg origin_name)" />
   <joint name="$(arg prefix)/$(arg origin_name)_fixed_joint" type="fixed">
     <parent link="$(arg origin_name)" />
